File: MCU_Board_V2/MCU_Board_V2.kicad_pcb (KiCad board)
At the start: 6 copper layers, 26 x 25 mm, 65 parts, among them IC3 AP62200WU-7, J1 USB_C_Receptacle_USB2.0, J2 DF12NB_5.0_-40DP-0.5V_51_, J3 DF12NB-40DS-0.5V_51_, J4 DF12NB-40DS-0.5V_51_, J5 DF12NB_5.0_-40DP-0.5V_51_, U4 USBLC6-2SC6, U5 STM32H723VGTx, U6 ZD25WQ32C, X1 F322516MUBCE2O

Commit message: Adjusted for JLC as manufacturer
Routing:
- net QSPI_IO0: track 11.3 -> 7.29 mm
- net +5V: track 44.5 -> 41.2 mm
- net USB_D+: track 8.74 -> 7.91 mm
- net USB_D-: track 8.62 -> 7.91 mm
- net QSPI_CLK: track 9.73 -> 9.10 mm
Other:
- board text added: "Impedance adjusted to the JLC06161H-3313 Stackup"
